File: Polaris/Rocket.kicad_sch (KiCad schematic)
At the start: 38 parts, among them J1 IMU_INT, SW1 SW_MEC_5E, U1 STM32H755XIHx, U2 HT75xx-1-SOT89

Commit message: Add files via upload
Parts:
- removed Barometer2: MS5611-01BA, Package_LGA:LGA-8_3x5mm_P1.25mm, symbol Sensor_Pressure:MS5611-01BA
- added C26, C29, C30: 100nF, Capacitor_SMD:C_0402_1005Metric, symbol Device:C
- added C27: 10uF, Capacitor_SMD:C_0201_0603Metric_Pad0.64x0.40mm_HandSolder, symbol Device:C
- added C28: 10uF, Capacitor_SMD:C_0402_1005Metric, symbol Device:C
- added D3: PMEG050V150EPD, Package_TO_SOT_SMD:Nexperia_CFP15_SOT-1289, symbol Diode:PMEG050V150EPD
- added D4: LED, LED_THT:LED_D3.0mm_Horizontal_O6.35mm_Z10.0mm, symbol Device:LED
- added IMU2: ISM330DHCX, Package_LGA:LGA-14_3x2.5mm_P0.5mm_LayoutBorder3x4y, symbol Sensor_Motion:ISM330DHCX
- added J2: IMU_INT, Connector_Wire:SolderWire-1sqmm_1x02_P5.4mm_D1.4mm_OD2.7mm, symbol Connector:Conn_01x02_Pin
- added R2: 510Ohm, Resistor_SMD:R_0201_0603Metric, symbol Device:R
- added U3: uA7808, Package_TO_SOT_THT:TO-220-3_Vertical, symbol Regulator_Linear:uA7808
- added U4: SST25VF080B-50-4x-S2Ax, Package_SO:SOIC-8_5.275x5.275mm_P1.27mm, symbol Memory_Flash:SST25VF080B-50-4x-S2Ax
- added U6: RFM69HCW, RF_Module:HOPERF_RFM9XW_SMD, symbol RF_Module:RFM69HCW
- added U7: NEO-M8M, RF_GPS:ublox_NEO, symbol RF_GPS:NEO-M8M
Connections:
- net 8V: now also C28.1, D4.2 (A), U3.3 (OUT)
- net Baro1CLK: now also U1.A13 (PC10); no longer U1.U14 (PB13)
- net Baro1MISO: now also U1.B13 (PC11); no longer U1.U15 (PB14)
- net Baro1MOSI: now also U1.R6 (PB2); no longer U1.T15 (PB15)
- net Baro1NSS: no longer U1.D15 (PA9)
- net GND: now also C26.2, C27.2, C28.2, C29.2, C30.2, IMU2.6 (GND), IMU2.7 (GND), R2.2, U3.2 (GND), U4.4 (VSS), U6.1 (GND), U6.10 (GND), U6.8 (GND), U7.10 (GND), U7.12 (GND), U7.13 (GND), U7.2 (D_SEL), U7.24 (GND)
- net SD1CLK: no longer U1.R6 (PB2)
- net SD1CS: no longer U1.E15 (PA8)
- net SD1MISO: no longer U1.C6 (PB3)
- net SD1MOSI: no longer U1.B7 (PB4)
- net Servo1PWM: now also U1.P9 (PE9); no longer U1.N4 (PA1)
- net Servo2PWM: now also U1.P10 (PE11); no longer U1.N3 (PA2)
- net VDD: now also C26.1, C29.1, C30.1, IMU2.5 (VDDIO), IMU2.8 (VDD), U4.8 (VDD), U6.13 (3.3V), U7.22 (V_BCKP), U7.23 (VCC)
- net RESET_N: now reaches C3.1, SW1.3 (K), SW1.4 (A), U1.K1 (NRST)
- net RESET_N: now also U7.8 (~{RESET})
- net MemoCLK: now reaches U1.C3 (PE2)
- net MemoCLK: now also U4.6 (SCK)
- net Radio_MISO: now reaches U1.C9 (PG12)
- net Radio_MISO: now also U6.2 (MISO)
- net MemoMISO: now reaches U1.D1 (PE5)
- net MemoMISO: now also U4.2 (SO)
- net Radio_MOSI: now reaches U1.D8 (PG14)
- net Radio_MOSI: now also U6.3 (MOSI)
- net Radio_CLK: now reaches U1.D9 (PG13)
- net Radio_CLK: now also U6.4 (SCK)
- net MemoMOSI: now reaches U1.E5 (PE6)
- net MemoMOSI: now also U4.5 (SI)
- net IMUCLK_1: now reaches U1.K3 (PF7)
- net IMUCLK_1: now also IMU1.13 (SCL)
- net IMUMISO_1: now reaches U1.K4 (PF8)
- net IMUMISO_1: now also IMU1.1 (SDO/SA0)
- net IMUMOSI_1: now reaches U1.L4 (PF9)
- net IMUMOSI_1: now also IMU1.14 (SDA)
- net IMUMOSI_2: now reaches U1.M2 (PC1)
- net IMUMOSI_2: now also IMU2.14 (SDA)
- net IMUCLK_2: now reaches U1.P11 (PB10)
- net IMUCLK_2: now also IMU2.13 (SCL)
- net IMUMISO_2: now reaches U1.R1 (PC2_C)
- net IMUMISO_2: now also IMU2.1 (SDO/SA0)
- net +5V renamed +3.8V
- net Baro2CLK renamed GPS_CLK
- net GPS_CLK: now also U7.19 (SCL/SPI_CLK)
- net Baro2MISO renamed GPS_MISO
- net GPS_MISO: now also U7.20 (TXD/SPI_MISO)
- net Baro2MOSI renamed GPS_MOSI
- net GPS_MOSI: now also U7.21 (RXD/SPI_MOSI)
- net Baro2NSS: no longer names the net of U1.U3 (PA4)
- removed net IMUCLK: IMU1.13 (SCL), U1.A13 (PC10)
- net IMUCS: no longer names the net of U1.A14 (PA15)
- net IMUCS: no longer IMU1.12 (CS)
- removed net IMUMISO: IMU1.1 (SDO/SA0), U1.B13 (PC11)
- net IMUMOSI: no longer names the net of U1.C12 (PC12)
- net IMUMOSI: no longer IMU1.14 (SDA)
- new net: IMU2.4 (INT1), J2.1 (Pin_1)
- new net: IMU2.9 (INT2), J2.2 (Pin_2)
- new net: D4.1 (K), R2.1
- new net: C27.1, D3.3 (K), U3.1 (IN)
- new net +10.8V: D3.1 (A), D3.2 (A)
- new net GPS_CS: U7.18 (SDA/~{SPI_CS})
- new net IMUCS_1: IMU1.12 (CS)
- new net IMUCS_2: IMU2.12 (CS)
- new net MemoCS: U4.1 (~{CE})
- new net Radio_CS: U6.5 (NSS)
Other:
- note added: "Polaris_Design_01"
- moved on the sheet: C1, C2, D1, D2, R1, SD1, Servo1, Servo2, U2

Commit message: Add files via upload
Parts:
- removed D1, D3: PMEG050V150EPD, Package_TO_SOT_SMD:Nexperia_CFP15_SOT-1289, symbol Diode:PMEG050V150EPD
- removed SD1: Conn_01x09_Pin, Connector_Hirose:Hirose_DF13-09P-1.25DSA_1x09_P1.25mm_Vertical, symbol Connector:Conn_01x09_Pin
- added J3: Micro_SD_Card, symbol Connector:Micro_SD_Card
Connections:
- net +3.8V: now also C1.1, U2.2 (VIN)
- net Baro1NSS: now also U1.C12 (PC12)
- net GND: now also J3.6 (VSS), J3.9 (SHIELD)
- net GPS_CS: now also U1.U3 (PA4)
- net IMUCS_1: now also U1.K2 (PF6)
- net IMUCS_2: now also U1.R2 (PC3_C)
- net MemoCS: now also U1.D2 (PE4)
- net Radio_CS: now also U1.B9 (PG11)
- net VDD: now also J3.4 (VDD)
- net at C5.1, C6.1, U1.A7 (VCAP): no longer U1.D17 (VCAP), U1.U11 (VCAP)
- net SD_CMD: now reaches U1.A14 (PA15)
- net SD_CMD: now also J3.3 (CMD)
- net SD_DATA3: now reaches U1.B14 (PA14)
- net SD_DATA3: now also J3.2 (DAT3/CD)
- net SD_DATA2: now reaches U1.C15 (PA13)
- net SD_DATA2: now also J3.1 (DAT2)
- net SD_DATA1: now reaches U1.E16 (PA12)
- net SD_DATA1: now also J3.8 (DAT1)
- net SD_DATA0: now reaches U1.E17 (PA11)
- net SD_DATA0: now also J3.7 (DAT0)
- net SD_CLK: now reaches U1.T10 (PE13)
- net SD_CLK: now also J3.5 (CLK)
- net +8.7V: now reaches C27.1, U3.1 (IN)
- no-connect marks 0 -> 172
